Commit message: feat(arcor2_ur): vgc10 attached to the robot

File: src/python/arcor2_ur/data/urdf/ur5e.urdf (robot description, URDF)
Before this commit: robot ur5e, 13 links, 12 joints
Links:
- added link onrobot_vgc10_base_link, mass 0.6; collision mesh filename=package://meshes/collision/base_link_1cup.stl; visual mesh filename=package://meshes/visual/base_link_1cup.stl
- added link suction, mass 0.2; collision mesh filename=package://meshes/collision/suction_cup_1cup.stl; visual mesh filename=package://meshes/visual/suction_cup_1cup.stl
Joints:
- added joint _suction_joint: type fixed, parent onrobot_vgc10_base_link, child suction, origin xyz=0 0 0.094901 rpy=0 0 0, axis 1 0 0
- added joint tool0-suction: type fixed, parent tool0, child onrobot_vgc10_base_link, origin xyz=0 0 0 rpy=0 0 0
